File: STM32F4X.sch (KiCad schematic (older format))
At the start: 92 parts, among them J1 POW_IN, J10 T2, J11 TC, J12 T3, J2 USB_B_Micro, J3 SWD_Conn, J4 Micro_SD_Card, J5 T0, J6 UART header, J7 TB, J8 T1, J9 SPI header 10pin, SW1 SW_SPDT, SW2 SW_RESET, U1 AOZ1282CI, U2 STM32F407VETx, U3 USBLC6-2SC6, Y1 16MHz-NX3225SA

Commit message: Added new checklist for hardware support. It will serve as the base for documentation! 	new file:   hardware_chklist.md
Parts:
- removed A?: DRV8825_X, Module:Pololu_Breakout-16_15.2x20.3mm, symbol Driver_Motor:Pololu_Breakout_DRV8825
- removed A?: A4988_Y, Module:Pololu_Breakout-16_15.2x20.3mm, symbol Driver_Motor:Pololu_Breakout_A4988
- removed A?: Pololu_Breakout_TMC2209, Module:Pololu_Breakout-16_15.2x20.3mm, symbol Trinamic_breakout:Pololu_Breakout_TMC2209
- removed A?: Pololu_Breakout_TMC2130, Module:Pololu_Breakout-16_15.2x20.3mm, symbol Trinamic_breakout:Pololu_Breakout_TMC2130
- removed C? (x3): 100uF, 65V, symbol Device:CP_Small
- removed J? (x3): Motor, symbol Connector:Conn_01x04_Female
- removed R? (x3): 10K, Resistor_SMD:R_0805_2012Metric_Pad1.20x1.40mm_HandSolder, symbol Device:R_Small
- added A1: DRIVER_X, Module:Pololu_Breakout-16_15.2x20.3mm, symbol Stepper_driver_generic_breakout:Motor_driver_generic_breakout
- added J13: Conn_01x04_Female, symbol Connector:Conn_01x04_Female
- added JP1: JMX1, symbol Jumper:Jumper_3_Open
- added JP2: JMX2, symbol Jumper:Jumper_3_Open
- added JP3: JMX3, symbol Jumper:Jumper_3_Open
- added JP?: JMX4, symbol Jumper:Jumper_3_Open
- added R25: 10k, Resistor_SMD:R_0805_2012Metric_Pad1.20x1.40mm_HandSolder, symbol Device:R_Small
- J2: symbol STM32F4X-rescue:USB_B_Micro-Connector -> STM32F4X-rescue:USB_B_Micro-Connector-STM32F4X-rescue
- U3: symbol STM32F4X-rescue:USBLC6-2SC6-Power_Protection -> STM32F4X-rescue:USBLC6-2SC6-Power_Protection-STM32F4X-rescue
- gave numbers to parts that had none: 3
Connections:
- net labels added: ENBL, MX1, MX2, MX3, PWM_BED, PWM_T0, PWM_T1, PWM_T2, PWM_T3, SDO_XT, SERVO1, SERVO2, SERVO3, SERVO4
- net labels removed: CS, MS0_X, MS0_Y, MS1_X, MS1_Y, MS2_X, MS2_Y, mMISO, mMOSI, mSCK
- wire segments 353 -> 322
- no-connect marks 10 -> 6

Commit message: Added all seven stepper drivers. Cube MX report for pin map.
Parts:
- removed JP?: JMX4, symbol Jumper:Jumper_3_Open
- added A2: DRIVER_6, Module:Pololu_Breakout-16_15.2x20.3mm, symbol Stepper_driver_generic_breakout:Motor_driver_generic_breakout
- added A3: DRIVER_5, Module:Pololu_Breakout-16_15.2x20.3mm, symbol Stepper_driver_generic_breakout:Motor_driver_generic_breakout
- added A4: DRIVER_4, Module:Pololu_Breakout-16_15.2x20.3mm, symbol Stepper_driver_generic_breakout:Motor_driver_generic_breakout
- added A5: DRIVER_2, Module:Pololu_Breakout-16_15.2x20.3mm, symbol Stepper_driver_generic_breakout:Motor_driver_generic_breakout
- added A6: DRIVER_3, Module:Pololu_Breakout-16_15.2x20.3mm, symbol Stepper_driver_generic_breakout:Motor_driver_generic_breakout
- added A?: DRIVER_7, Module:Pololu_Breakout-16_15.2x20.3mm, symbol Stepper_driver_generic_breakout:Motor_driver_generic_breakout
- added C28, C29, C30, C31, C32, C33, C?: 100uF, 65V, symbol Device:CP_Small
- added J14, J15, J16, J23, J24, J?: Conn_01x04_Female, symbol Connector:Conn_01x04_Female
- added J17: X_MIN, symbol Connector:Conn_01x03_Male
- added J18: X_MAX, symbol Connector:Conn_01x03_Male
- added J19: Y_MIN, symbol Connector:Conn_01x03_Male
- added J20: Y_MAX, symbol Connector:Conn_01x03_Male
- added J21: Z_MIN, symbol Connector:Conn_01x03_Male
- added J22: Z_MAX, symbol Connector:Conn_01x03_Male
- added JP10, JP14, JP16, JP18, JP5, JP?: JMX2, symbol Jumper:Jumper_3_Open
- added JP11, JP19, JP20, JP21, JP6, JP?: JMX3, symbol Jumper:Jumper_3_Open
- added JP12, JP22, JP23, JP24, JP7, JP8, JP?: JMX4, symbol Jumper:Jumper_3_Open
- added JP13, JP15, JP17, JP4, JP9, JP?: JMX1, symbol Jumper:Jumper_3_Open
- added R26, R27, R28, R29, R30, R31, R34, R35, R36, R37, R38, R40, R41, R42, R43, R44, R45, R46, R47, R48, R49, R52, R53, R54, R? (x4): 100E, symbol Device:R_Small
- added R32, R33, R39, R50, R51, R?: 10k, Resistor_SMD:R_0805_2012Metric_Pad1.20x1.40mm_HandSolder, symbol Device:R_Small
- added RN1, RN2, RN3, RN4, RN5, RN6, RN?: 100E, symbol Device:R_Pack03
- A1: value DRIVER_X -> DRIVER_1
Connections:
- net +3V3: now also A2.2 (VCC_IO/~FLT), A3.2 (VCC_IO/~FLT), A4.2 (VCC_IO/~FLT), A5.2 (VCC_IO/~FLT), A6.2 (VCC_IO/~FLT), A?.2 (VCC_IO/~FLT), J17.1 (Pin_1), J18.1 (Pin_1), J19.1 (Pin_1), J20.1 (Pin_1), J21.1 (Pin_1), J22.1 (Pin_1), JP10.3 (B), JP11.3 (B), JP12.3 (B), JP13.3 (B), JP14.3 (B), JP15.3 (B), JP16.3 (B), JP17.3 (B), JP18.3 (B), JP19.3 (B), JP20.3 (B), JP21.3 (B), JP22.3 (B), JP23.3 (B), JP24.3 (B), JP4.3 (B), JP5.3 (B), JP6.3 (B), JP7.3 (B), JP8.3 (B), JP9.3 (B), JP?.3 (B), JP?.3 (B), JP?.3 (B), JP?.3 (B), R32.1, R33.1, R39.1, R50.1, R51.1, R?.1
- net GND1: now also A2.1 (GND), A2.7 (GND), A3.1 (GND), A3.7 (GND), A4.1 (GND), A4.7 (GND), A5.1 (GND), A5.7 (GND), A6.1 (GND), A6.7 (GND), A?.1 (GND), A?.7 (GND), C28.2, C29.2, C30.2, C31.2, C32.2, C33.2, C?.2, J17.2 (Pin_2), J18.2 (Pin_2), J19.2 (Pin_2), J20.2 (Pin_2), J21.2 (Pin_2), J22.2 (Pin_2)
- net SPI2_CS: no longer JP3.1 (A)
- net SPI2_MISO: now also R34.2, R35.2, R40.2, R52.2, R53.2, R54.2, R?.2
- net SPI2_MOSI: now also R26.2, R29.2, R36.2, R41.2, R43.2, R45.2, R?.2; no longer JP1.1 (A)
- net SPI2_SCK: now also R27.2, R30.2, R37.2, R42.2, R44.2, R46.2, R?.2; no longer JP2.1 (A)
- net SPI_CS: no longer U2.29 (PA4)
- net UART4_RX: now also J6.1 (Pin_1)
- net UART4_TX: now also J6.2 (Pin_2)
- net USART2_TX: now also R47.2
- net VCC: now also A1.8 (VMOT), A2.8 (VMOT), A3.8 (VMOT), A4.8 (VMOT), A5.8 (VMOT), A6.8 (VMOT), A?.8 (VMOT), C28.1, C29.1, C30.1, C31.1, C32.1, C33.1, C?.1
- net E_STOP_XMAX: now reaches U2.1 (PE2)
- net E_STOP_XMAX: now also J18.3 (Pin_3)
- net E_STOP_YMIN: now reaches U2.2 (PE3)
- net E_STOP_YMIN: now also J19.3 (Pin_3)
- net E_STOP_YMAX: now reaches U2.3 (PE4)
- net E_STOP_YMAX: now also J20.3 (Pin_3)
- net E_STOP_ZMIN: now reaches U2.4 (PE5)
- net E_STOP_ZMIN: now also J21.3 (Pin_3)
- net USART3_TX: now reaches U2.47 (PB10)
- net USART3_TX: now also R48.2
- net E_STOP_ZMAX: now reaches U2.5 (PE6)
- net E_STOP_ZMAX: now also J22.3 (Pin_3)
- net USART1_TX: now reaches U2.68 (PA9)
- net USART1_TX: now also R49.2
- net E_STOP_XMIN: now reaches U2.98 (PE1)
- net E_STOP_XMIN: now also J17.3 (Pin_3)
- net DIR renamed 1DRV-DIR
- net 1DRV-DIR: now also RN4.4 (R3.2)
- net ENBL renamed 1DRV-EN
- net 1DRV-EN: now also RN4.6 (R1.2)
- net MX1 renamed 1MX1
- net 1MX1: now also JP13.2 (C); no longer JP1.2 (C)
- net MX2 renamed 1MX2
- net 1MX2: now also JP14.2 (C); no longer JP2.2 (C)
- net MX3 renamed 1MX3
- net 1MX3: now also JP21.2 (C); no longer JP3.2 (C)
- net SDO_XT renamed 1SDO_XT
- net 1SDO_XT: now also JP22.2 (C)
- net STEP renamed 1DRV-STP
- net 1DRV-STP: now also RN4.5 (R2.2)
- net USART2_RX: no longer names the net of U2.26 (PA3)
- net USART_RX: no longer names the net of U2.56 (PD9)
- net USART_RX: no longer J6.1 (Pin_1)
- net USART_TX: no longer names the net of U2.55 (PD8)
- net USART_TX: no longer J6.2 (Pin_2)
- new net: A6.3 (A2), J24.4 (Pin_4)
- new net: A6.4 (A1), J24.3 (Pin_3)
- new net: A6.5 (B1), J24.2 (Pin_2)
- new net: A6.6 (B2), J24.1 (Pin_1)
- new net: A4.3 (A2), J16.4 (Pin_4)
- new net: A4.4 (A1), J16.3 (Pin_3)
- new net: A4.5 (B1), J16.2 (Pin_2)
- new net: A4.6 (B2), J16.1 (Pin_1)
- new net: A3.3 (A2), J15.4 (Pin_4)
- new net: A3.4 (A1), J15.3 (Pin_3)
- new net: A3.5 (B1), J15.2 (Pin_2)
- new net: A3.6 (B2), J15.1 (Pin_1)
- new net: A2.3 (A2), J14.4 (Pin_4)
- new net: A2.4 (A1), J14.3 (Pin_3)
- new net: A2.5 (B1), J14.2 (Pin_2)
- new net: A2.6 (B2), J14.1 (Pin_1)
- new net: JP1.1 (A), R26.1
- new net: JP2.1 (A), R27.1
- new net: JP3.1 (A), R28.1
- new net: JP7.1 (A), R34.1
- new net: A5.3 (A2), J23.4 (Pin_4)
- new net: A5.4 (A1), J23.3 (Pin_3)
- new net: A5.5 (B1), J23.2 (Pin_2)
- new net: A5.6 (B2), J23.1 (Pin_1)
- new net: JP4.1 (A), R29.1
- new net: JP5.1 (A), R30.1
- new net: JP9.1 (A), R36.1
- new net: JP10.1 (A), R37.1
- new net: JP17.1 (A), R45.1
- new net: JP18.1 (A), R46.1
- new net: JP15.1 (A), R43.1
- new net: JP16.1 (A), R44.1
- new net: JP13.1 (A), R41.1
- new net: JP14.1 (A), R42.1
- new net: JP6.1 (A), R31.1
- new net: JP8.1 (A), R35.1
- new net: JP11.1 (A), R38.1
- new net: JP12.1 (A), R40.1
- new net: JP20.1 (A), R48.1
- new net: JP24.1 (A), R54.1
- new net: JP19.1 (A), R47.1
- new net: JP23.1 (A), R53.1
- new net: JP21.1 (A), R49.1
- new net: JP22.1 (A), R52.1
- new net: A?.3 (A2), J?.4 (Pin_4)
- new net: A?.4 (A1), J?.3 (Pin_3)
- new net: A?.5 (B1), J?.2 (Pin_2)
- new net: A?.6 (B2), J?.1 (Pin_1)
- new net: JP?.1 (A), R?.1 (x4)
- new net 1DIR: RN4.3 (R3.1)
- new net 1ENBL: RN4.1 (R1.1)
- new net 1STP: RN4.2 (R2.1)
- new net 2DIR: RN5.3 (R3.1)
- new net 2DRV-DIR: A5.16 (DIR), RN5.4 (R3.2)
- new net 2DRV-EN: A5.9 (~EN), A6.9 (~EN), R50.2, R51.2, RN5.6 (R1.2)
- new net 2DRV-STEP: A5.15 (STEP)
- new net 2DRV-STP: RN5.5 (R2.2)
- new net 2ENBL: RN5.1 (R1.1)
- new net 2MX1: A5.10 (M1/CFG1/SDI), JP15.2 (C)
- new net 2MX2: A5.11 (M2/CFG2/SCK), JP16.2 (C)
- new net 2MX3: A5.12 (M3/CFG3/CS/PDN), JP19.2 (C)
- new net 2SDO_XT: A5.13 (UART/SDO/CFG0/~RST), A5.14 (CLK/DCO/~SLP), JP23.2 (C)
- new net 2STP: RN5.2 (R2.1)
- new net 3DIR: RN6.3 (R3.1)
- new net 3DRV-DIR: A6.16 (DIR), RN6.4 (R3.2)
- new net 3DRV-EN: RN6.6 (R1.2)
- new net 3DRV-STEP: A6.15 (STEP)
- new net 3DRV-STP: RN6.5 (R2.2)
- new net 3ENBL: RN6.1 (R1.1)
- new net 3MX1: A6.10 (M1/CFG1/SDI), JP17.2 (C)
- new net 3MX2: A6.11 (M2/CFG2/SCK), JP18.2 (C)
- new net 3MX3: A6.12 (M3/CFG3/CS/PDN), JP20.2 (C)
- new net 3SDO_XT: A6.13 (UART/SDO/CFG0/~RST), A6.14 (CLK/DCO/~SLP), JP24.2 (C)
- new net 3STP: RN6.2 (R2.1)
- new net 4DIR: RN3.3 (R3.1)
- new net 4DRV-DIR: A4.16 (DIR), RN3.4 (R3.2)
- new net 4DRV-EN: A4.9 (~EN), R39.2, RN3.6 (R1.2)
- new net 4DRV-STEP: A4.15 (STEP)
- new net 4DRV-STP: RN3.5 (R2.2)
- new net 4ENBL: RN3.1 (R1.1)
- new net 4MX1: A4.10 (M1/CFG1/SDI), JP9.2 (C)
- new net 4MX2: A4.11 (M2/CFG2/SCK), JP10.2 (C)
- new net 4MX3: A4.12 (M3/CFG3/CS/PDN), JP11.2 (C)
- new net 4SDO_XT: A4.13 (UART/SDO/CFG0/~RST), A4.14 (CLK/DCO/~SLP), JP12.2 (C)
- new net 4STP: RN3.2 (R2.1)
- new net 5DIR: RN2.3 (R3.1)
- new net 5DRV-DIR: A3.16 (DIR), RN2.4 (R3.2)
- new net 5DRV-EN: A3.9 (~EN), R33.2, RN2.6 (R1.2)
- new net 5DRV-STEP: A3.15 (STEP)
- new net 5DRV-STP: RN2.5 (R2.2)
- new net 5ENBL: RN2.1 (R1.1)
- new net 5MX1: A3.10 (M1/CFG1/SDI), JP4.2 (C)
- new net 5MX2: A3.11 (M2/CFG2/SCK), JP5.2 (C)
- new net 5MX3: A3.12 (M3/CFG3/CS/PDN), JP6.2 (C)
- new net 5SDO_XT: A3.13 (UART/SDO/CFG0/~RST), A3.14 (CLK/DCO/~SLP), JP8.2 (C)
- new net 5STP: RN2.2 (R2.1)
- new net 6DIR: RN1.3 (R3.1)
- new net 6DRV-DIR: A2.16 (DIR), RN1.4 (R3.2)
- new net 6DRV-EN: A2.9 (~EN), R32.2, RN1.6 (R1.2)
- new net 6DRV-STEP: A2.15 (STEP)
- new net 6DRV-STP: RN1.5 (R2.2)
- new net 6ENBL: RN1.1 (R1.1)
- new net 6MX1: A2.10 (M1/CFG1/SDI), JP1.2 (C)
- new net 6MX2: A2.11 (M2/CFG2/SCK), JP2.2 (C)
- new net 6MX3: A2.12 (M3/CFG3/CS/PDN), JP3.2 (C)
- new net 6SDO_XT: A2.13 (UART/SDO/CFG0/~RST), A2.14 (CLK/DCO/~SLP), JP7.2 (C)
- new net 6STP: RN1.2 (R2.1)
- new net 7DIR: RN?.3 (R3.1)
- new net 7DRV-DIR: A?.16 (DIR), RN?.4 (R3.2)
- new net 7DRV-EN: A?.9 (~EN), R?.2, RN?.6 (R1.2)
- new net 7DRV-STEP: A?.15 (STEP)
- new net 7DRV-STP: RN?.5 (R2.2)
- new net 7ENBL: RN?.1 (R1.1)
- new net 7MX1: A?.10 (M1/CFG1/SDI), JP?.2 (C)
- new net 7MX2: A?.11 (M2/CFG2/SCK), JP?.2 (C)
- new net 7MX3: A?.12 (M3/CFG3/CS/PDN), JP?.2 (C)
- new net 7SDO_XT: A?.13 (UART/SDO/CFG0/~RST), A?.14 (CLK/DCO/~SLP), JP?.2 (C)
- new net 7STP: RN?.2 (R2.1)
- new net SPI2_CS4: R38.2
- new net SPI2_CS5: R31.2
- new net SPI2_CS6: R28.2
- new net SPI2_CS7: R?.2
Other:
- note added: "BLOCK B3: CHECK LDO FUNCTIONALITY. SEARCH ALTERNATIVES.\n"
- note added: "For stepper drivers, SPI based drivers will use the same SPI2 lines and different CS line for each driver.\nNow RX/TX based drivers like TMC2208, will use single wire UART through the same CS line.\nModify driver according to use PDN pin for UART.\n"
- note added: "Limit Switches"
- note added: "Place VMOT capacitor close to driver."
- moved on the sheet: A1, C17, C4, C5, J13, R11, R25, SW2, U2

Commit message: Finalized pin maps
Parts:
- gave numbers to parts that had none: 13
Connections:
- net 2DRV-STEP is gone; now on net 2DRV-STP: A5.15 (STEP)
- net 3DRV-STEP is gone; now on net 3DRV-STP: A6.15 (STEP)
- net 4DRV-STEP is gone; now on net 4DRV-STP: A4.15 (STEP)
- net 5DRV-STEP is gone; now on net 5DRV-STP: A3.15 (STEP)
- net 6DRV-STEP is gone; now on net 6DRV-STP: A2.15 (STEP)
- net 7DRV-STEP is gone; now on net 7DRV-STP: A7.15 (STEP)
- net SPI2_CS is gone; now on net SPI2_CS6: U2.53 (PB14)
- net 1DIR: now also U2.58 (PD11)
- net 1ENBL: now also U2.56 (PD9)
- net 1STP: now also U2.57 (PD10)
- net 2DIR: now also U2.7 (PC13)
- net 2DRV-EN: no longer A6.9 (~EN), R51.2
- net 2ENBL: now also U2.97 (PE0)
- net 2STP: now also U2.96 (PB9)
- net 3DIR: now also U2.8 (PC14)
- net 3DRV-EN: now also A6.9 (~EN), R51.2
- net 3ENBL: now also U2.88 (PD7)
- net 3STP: now also U2.95 (PB8)
- net 4DIR: now also U2.9 (PC15)
- net 4ENBL: now also U2.87 (PD6)
- net 4STP: now also U2.91 (PB5)
- net 5DIR: now also U2.85 (PD4)
- net 5ENBL: now also U2.82 (PD1)
- net 5STP: now also U2.90 (PB4)
- net 6DIR: now also U2.84 (PD3)
- net 6ENBL: now also U2.81 (PD0)
- net 6STP: now also U2.77 (PA15)
- net 7DIR: now also U2.38 (PE7)
- net 7ENBL: now also U2.29 (PA4)
- net 7STP: now also U2.26 (PA3)
- net SPI2_CS4: now also U2.51 (PB12)
- net SPI2_CS5: now also U2.48 (PB11)
- net SPI2_CS7: now also U2.55 (PD8)
- no-connect marks 6 -> 14
Other:
- note added: "PC7 IS AN EXTRA_PWM\nLEFT UNCONNECTED\nFOR FUTURE.\n"
- moved on the sheet: C17, C4, C5, R11, RN4, RN5, RN6, SW2, U2
